File: vsdsquadron_ai_1A/vsdsquadron_ai_1A.kicad_pcb (KiCad board)
At the start: 2 copper layers, 90 x 120 mm, 4 parts, among them U1 CAMERA-OV7670

Commit message: Fianl changes
Parts:
- added kibuzzard-66C8A791: G***, kibuzzard-66C8A791, F.Cu at (75.3, 113.0)
- added kibuzzard-66C8A791: G***, kibuzzard-66C8A791, F.Cu at (113.3, 113.0)
- added kibuzzard-66C8A7E0: G***, kibuzzard-66C8A7E0, F.Cu at (113.2, 121.0)
- added kibuzzard-66C8A86F: G***, kibuzzard-66C8A86F, F.Cu at (71.5, 126.5)
- added kibuzzard-66C8AD7B: G***, kibuzzard-66C8AD7B, F.Cu at (96.1, 54.1)
- added kibuzzard-66C8ADA8: G***, kibuzzard-66C8ADA8, F.Cu at (95.5, 165.5)
Connections:
- Camera_VSDMini1 pad 22: unconnected-(Camera_VSDMini1-+5V-Pad22) -> Net-(Camera_VSDMini1-+5V)
- Predictor_VSDMini1 pad 22: unconnected-(Predictor_VSDMini1-+5V-Pad22) -> Net-(Camera_VSDMini1-+5V)
Routing:
- net +3.3V: track 92.2 -> 0.00 mm, vias 1 -> 0
- net Net-(Camera_VSDMini1-+5V): track 0.00 -> 47.0 mm
- net GND: track 8.80 -> 21.3 mm, vias 1 -> 3
- net Net-(AFF1-a): track 36.3 -> 46.6 mm
- net Net-(Camera_VSDMini1-Nano_PC1): track 44.9 -> 49.8 mm
- net Net-(Camera_VSDMini1-Nano_PA2): track 43.3 -> 47.5 mm
- net Net-(Camera_VSDMini1-Nano_PC0): track 55.3 -> 59.0 mm, vias 0 -> 2
- net Net-(Camera_VSDMini1-Nano_PD2): track 49.8 -> 53.4 mm
- net Net-(Camera_VSDMini1-Nano_PD5): track 79.6 -> 82.8 mm, vias 0 -> 1
- net Net-(Camera_VSDMini1-Nano_PC5): track 102.9 -> 101.0 mm, vias 0 -> 2
- net Net-(Camera_VSDMini1-Nano_PC3): track 91.2 -> 89.7 mm, vias 0 -> 2
- net Net-(Camera_VSDMini1-Nano_PD3): track 41.9 -> 43.5 mm, vias 0 -> 1
- net Net-(Camera_VSDMini1-Nano_PD0): track 43.7 -> 45.2 mm
- net Net-(Camera_VSDMini1-Nano_PC6): track 66.8 -> 68.2 mm
- net Net-(Camera_VSDMini1-Nano_PC2): track 49.6 -> 50.7 mm
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Other:
- outline, holes or cut-outs redrawn

Commit message: Edited footprint
Connections:
- Camera_VSDMini1 pad 15: GND -> unconnected-(Camera_VSDMini1-D_SWCLK-Pad15)
- Camera_VSDMini1 pad 16: +3.3V -> unconnected-(Camera_VSDMini1-D_SWDIO-Pad16)
- Camera_VSDMini1 pad 17: unconnected-(Camera_VSDMini1-RST-Pad17) -> Net-(Camera_VSDMini1-Nano_PD5)
- Camera_VSDMini1 pad 19: Net-(Camera_VSDMini1-Nano_PD5) -> unconnected-(Camera_VSDMini1-RST-Pad19)
- Camera_VSDMini1 pad 20: unconnected-(Camera_VSDMini1-D_SWDIO-Pad20) -> +3.3V
- Camera_VSDMini1 pad 21: unconnected-(Camera_VSDMini1-D_SWCLK-Pad21) -> GND
- Predictor_VSDMini1 pad 15: GND -> unconnected-(Predictor_VSDMini1-D_SWCLK-Pad15)
- Predictor_VSDMini1 pad 16: +3.3V -> unconnected-(Predictor_VSDMini1-D_SWDIO-Pad16)
- Predictor_VSDMini1 pad 17: unconnected-(Predictor_VSDMini1-RST-Pad17) -> Net-(Predictor_VSDMini1-Nano_PD5)
- Predictor_VSDMini1 pad 19: Net-(Predictor_VSDMini1-Nano_PD5) -> unconnected-(Predictor_VSDMini1-RST-Pad19)
- Predictor_VSDMini1 pad 20: unconnected-(Predictor_VSDMini1-D_SWDIO-Pad20) -> +3.3V
- Predictor_VSDMini1 pad 21: unconnected-(Predictor_VSDMini1-D_SWCLK-Pad21) -> GND
Routing:
- net Net-(Camera_VSDMini1-Nano_PD5): track 82.8 -> 92.3 mm
- net Net-(Predictor_VSDMini1-Nano_PD5): track 24.8 -> 26.5 mm
Changed lines of the file:
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@@
 	(net 8 "Net-(AFF1-g)")
 	(net 9 "unconnected-(AFF1-DP-Pad5)")
-	(net 10 "unconnected-(Camera_VSDMini1-RST-Pad17)")
+	(net 10 "unconnected-(Camera_VSDMini1-RST-Pad19)")
 	(net 11 "Net-(Camera_VSDMini1-Nano_PC7)")
 	(net 12 "unconnected-(Camera_VSDMini1-Nano_PD6-Pad1)")
@@
 	(net 21 "Net-(Camera_VSDMini1-Nano_PA1)")
 	(net 22 "Net-(Camera_VSDMini1-Nano_PC1)")
-	(net 23 "unconnected-(Camera_VSDMini1-D_SWCLK-Pad21)")
+	(net 23 "unconnected-(Camera_VSDMini1-D_SWDIO-Pad16)")
 	(net 24 "unconnected-(Camera_VSDMini1-Nano_PD1-Pad24)")
 	(net 25 "Net-(Camera_VSDMini1-Nano_PD0)")
@@
 	(net 28 "Net-(Camera_VSDMini1-Nano_PC5)")
 	(net 29 "Net-(Camera_VSDMini1-Nano_PC0)")
-	(net 30 "unconnected-(Camera_VSDMini1-D_SWDIO-Pad20)")
+	(net 30 "unconnected-(Camera_VSDMini1-D_SWCLK-Pad15)")
 	(net 31 "Net-(Camera_VSDMini1-Nano_PC3)")
 	(net 32 "Net-(Camera_VSDMini1-Nano_PD2)")
@@
 	(net 35 "unconnected-(Predictor_VSDMini1-Nano_PD7-Pad2)")
 	(net 36 "Net-(Predictor_VSDMini1-Nano_PD5)")
-	(net 37 "unconnected-(Predictor_VSDMini1-D_SWCLK-Pad21)")
+	(net 37 "unconnected-(Predictor_VSDMini1-D_SWCLK-Pad15)")
 	(net 38 "unconnected-(Predictor_VSDMini1-Nano_PA1-Pad3)")
 	(net 39 "unconnected-(Predictor_VSDMini1-Nano_PD4-Pad27)")
 	(net 40 "unconnected-(Predictor_VSDMini1-Nano_PD1-Pad24)")
 	(net 41 "unconnected-(Predictor_VSDMini1-TX-Pad18)")
-	(net 42 "unconnected-(Predictor_VSDMini1-D_SWDIO-Pad20)")
+	(net 42 "unconnected-(Predictor_VSDMini1-D_SWDIO-Pad16)")
 	(net 43 "unconnected-(Predictor_VSDMini1-Nano_PD0-Pad7)")
 	(net 44 "unconnected-(Predictor_VSDMini1-Nano_PC7-Pad23)")
-	(net 45 "unconnected-(Predictor_VSDMini1-RST-Pad17)")
+	(net 45 "unconnected-(Predictor_VSDMini1-RST-Pad19)")
 	(net 46 "unconnected-(Predictor_VSDMini1-Nano_PA2-Pad4)")
 	(net 47 "unconnected-(Predictor_VSDMini1-Nano_PD2-Pad25)")
@@
 				(font
 					(size 0.001 0.001)
+					(thickness 0.15)
 				)
 			)
@@
 				(font
 					(size 0.001 0.001)
+					(thickness 0.15)
 				)
 			)
@@
 		(fp_arc
 			(start 34.156433 -12.163567)
-			(mid 35.570643 -11.577796)
+			(mid 35.570678 -11.577802)
 			(end 36.156433 -10.163567)
 			(stroke
@@
 			(layers "*.Cu" "*.Mask")
 			(remove_unused_layers no)
-			(net 20 "GND")
-			(pinfunction "GND")
-			(pintype "power_out")
+			(net 37 "unconnected-(Predictor_VSDMini1-D_SWCLK-Pad15)")
+			(pinfunction "D_SWCLK")
+			(pintype "input")
 		)
 		(pad "16" thru_hole oval
@@
 			(layers "*.Cu" "*.Mask")
 			(remove_unused_layers no)
-			(net 5 "+3.3V")
-			(pinfunction "+3.3V")
-			(pintype "power_in")
+			(net 42 "unconnected-(Predictor_VSDMini1-D_SWDIO-Pad16)")
+			(pinfunction "D_SWDIO")
+			(pintype "input")
 		)
 		(pad "17" thru_hole oval
@@
 			(layers "*.Cu" "*.Mask")
 			(remove_unused_layers no)
-			(net 45 "unconnected-(Predictor_VSDMini1-RST-Pad17)")
-			(pinfunction "RST")
+			(net 36 "Net-(Predictor_VSDMini1-Nano_PD5)")
+			(pinfunction "RX")
 			(pintype "input")
 		)
@@
 			(layers "*.Cu" "*.Mask")
 			(remove_unused_layers no)
-			(net 36 "Net-(Predictor_VSDMini1-Nano_PD5)")
-			(pinfunction "RX")
+			(net 45 "unconnected-(Predictor_VSDMini1-RST-Pad19)")
+			(pinfunction "RST")
 			(pintype "input")
 		)
@@
 			(layers "*.Cu" "*.Mask")
 			(remove_unused_layers no)
-			(net 42 "unconnected-(Predictor_VSDMini1-D_SWDIO-Pad20)")
-			(pinfunction "D_SWDIO")
-			(pintype "input")
+			(net 5 "+3.3V")
+			(pinfunction "+3.3V")
+			(pintype "power_in")
 		)
 		(pad "21" thru_hole rect
@@
 			(layers "*.Cu" "*.Mask")
 			(remove_unused_layers no)
-			(net 37 "unconnected-(Predictor_VSDMini1-D_SWCLK-Pad21)")
-			(pinfunction "D_SWCLK")
-			(pintype "input")
+			(net 20 "GND")
+			(pinfunction "GND")
+			(pintype "power_out")
 		)
 		(pad "22" thru_hole rect
@@
 				(font
 					(size 0.001 0.001)
+					(thickness 0.15)
 				)
 			)
@@
 				(font
 					(size 0.001 0.001)
+					(thickness 0.15)
 				)
 			)
@@
 				(font
 					(size 0.001 0.001)
+					(thickness 0.15)
 				)
 			)
@@
 				(font
 					(size 0.001 0.001)
+					(thickness 0.15)
 				)
 			)
@@
 		(fp_arc
 			(start 34.156433 -12.163567)
-			(mid 35.570643 -11.577796)
+			(mid 35.570678 -11.577802)
 			(end 36.156433 -10.163567)
 			(stroke
@@
 			(layers "*.Cu" "*.Mask")
 			(remove_unused_layers no)
-			(net 20 "GND")
-			(pinfunction "GND")
-			(pintype "power_out")
+			(net 30 "unconnected-(Camera_VSDMini1-D_SWCLK-Pad15)")
+			(pinfunction "D_SWCLK")
+			(pintype "input")
 		)
 		(pad "16" thru_hole oval
@@
 			(layers "*.Cu" "*.Mask")
 			(remove_unused_layers no)
-			(net 5 "+3.3V")
-			(pinfunction "+3.3V")
-			(pintype "power_in")
+			(net 23 "unconnected-(Camera_VSDMini1-D_SWDIO-Pad16)")
+			(pinfunction "D_SWDIO")
+			(pintype "input")
 		)
 		(pad "17" thru_hole oval
@@
 			(layers "*.Cu" "*.Mask")
 			(remove_unused_layers no)
-			(net 10 "unconnected-(Camera_VSDMini1-RST-Pad17)")
-			(pinfunction "RST")
+			(net 18 "Net-(Camera_VSDMini1-Nano_PD5)")
+			(pinfunction "RX")
 			(pintype "input")
 		)
@@
 			(layers "*.Cu" "*.Mask")
 			(remove_unused_layers no)
-			(net 18 "Net-(Camera_VSDMini1-Nano_PD5)")
-			(pinfunction "RX")
+			(net 10 "unconnected-(Camera_VSDMini1-RST-Pad19)")
+			(pinfunction "RST")
 			(pintype "input")
 		)
@@
 			(layers "*.Cu" "*.Mask")
 			(remove_unused_layers no)
-			(net 30 "unconnected-(Camera_VSDMini1-D_SWDIO-Pad20)")
-			(pinfunction "D_SWDIO")
-			(pintype "input")
+			(net 5 "+3.3V")
+			(pinfunction "+3.3V")
+			(pintype "power_in")
 		)
 		(pad "21" thru_hole rect
@@
 			(layers "*.Cu" "*.Mask")
 			(remove_unused_layers no)
-			(net 23 "unconnected-(Camera_VSDMini1-D_SWCLK-Pad21)")
-			(pinfunction "D_SWCLK")
-			(pintype "input")
+			(net 20 "GND")
+			(pinfunction "GND")
+			(pintype "power_out")
 		)
 		(pad "22" thru_hole rect
@@
 				(font
 					(size 0.001 0.001)
+					(thickness 0.15)
 				)
 			)
@@
 				(font
 					(size 0.001 0.001)
+					(thickness 0.15)
 				)
 			)
@@
 				(font
 					(size 0.001 0.001)
+					(thickness 0.15)
 				)
 			)
@@
 				(font
 					(size 0.001 0.001)
+					(thickness 0.15)
 				)
 			)
@@
 	)
 	(segment
-		(start 103.985033 102.214967)
-		(end 101.025033 102.214967)
-		(width 0.5)
+		(start 106.3 102.2)
+		(end 106.285033 102.214967)
+		(width 0.508)
 		(layer "F.Cu")
 		(net 18)
 	)
 	(segment
-		(start 106.2 100)
-		(end 103.985033 102.214967)
-		(width 0.5)
+		(start 106.285033 102.214967)
+		(end 101.025033 102.214967)
+		(width 0.508)
 		(layer "F.Cu")
 		(net 18)
 	)
 	(via
-		(at 106.2 100)
+		(at 106.3 102.2)
 		(size 1)
 		(drill 0.6)
@@
 	)
 	(segment
-		(start 110.58 95.62)
-		(end 110.58 82.5)
-		(width 0.5)
+		(start 115 80.1)
+		(end 115.660033 80.760033)
+		(width 0.508)
 		(layer "B.Cu")
 		(net 18)
 	)
 	(segment
-		(start 110.58 82.5)
-		(end 110.580033 82.499967)
-		(width 0.5)
+		(start 115.660033 82.499967)
+		(end 115.660033 92.839967)
+		(width 0.508)
 		(layer "B.Cu")
 		(net 18)
 	)
 	(segment
-		(start 110.580033 82.499967)
-		(end 110.580033 82.296392)
-		(width 0.5)
+		(start 115.660033 92.839967)
+		(end 106.3 102.2)
+		(width 0.508)
 		(layer "B.Cu")
 		(net 18)
 	)
 	(segment
-		(start 110.580033 82.296392)
-		(end 108.483641 80.2)
-		(width 0.5)
+		(start 115.660033 80.760033)
+		(end 115.660033 82.499967)
+		(width 0.508)
 		(layer "B.Cu")
 		(net 18)
 	)
 	(segment
-		(start 108.483641 80.2)
-		(end 90.8 80.2)
-		(width 0.5)
+		(start 67.765033 103.28071)
+		(end 90.945743 80.1)
+		(width 0.508)
 		(layer "B.Cu")
 		(net 18)
 	)
 	(segment
-		(start 106.2 100)
-		(end 110.58 95.62)
-		(width 0.5)
+		(start 90.945743 80.1)
+		(end 115 80.1)
+		(width 0.508)
 		(layer "B.Cu")
 		(net 18)
 	)
 	(segment
-		(start 90.8 80.2)
-		(end 67.765 103.235)
-		(width 0.5)
-		(layer "B.Cu")
-		(net 18)
-	)
-	(segment
-		(start 67.765 103.235)
-		(end 67.765 107.2)
-		(width 0.5)
+		(start 67.765033 107.199967)
+		(end 67.765033 103.28071)
+		(width 0.508)
 		(layer "B.Cu")
 		(net 18)
@@
 	)
 	(segment
-		(start 72.84 95.1017)
-		(end 72.84 83)
-		(width 0.5)
-		(layer "F.Cu")
+		(start 77.920033 82.999967)
+		(end 77.920033 89.282048)
+		(width 0.508)
+		(layer "B.Cu")
 		(net 36)
 	)
 	(segment
-		(start 65.2267 102.715)
-		(end 72.84 95.1017)
-		(width 0.5)
-		(layer "F.Cu")
+		(start 77.920033 89.282048)
+		(end 64.487114 102.714967)
+		(width 0.508)
+		(layer "B.Cu")
 		(net 36)
 	)
 	(segment
-		(start 63.285 102.715)
-		(end 65.2267 102.715)
-		(width 0.5)
-		(layer "F.Cu")
+		(start 64.487114 102.714967)
+		(end 63.285033 102.714967)
+		(width 0.508)
+		(layer "B.Cu")
 		(net 36)
 	)
