File: vsdsquadron_ai_1A/vsdsquadron_ai_1A.kicad_sch (KiCad schematic)
At the start: 4 parts, among them U1 CAMERA-OV7670

Commit message: Fianl changes
Connections:
- net at Camera_VSDMini1.22 (+5V): now also Predictor_VSDMini1.22 (+5V)
Changed lines of the file:
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@@
+	(wire
+		(pts
+			(xy 229.87 26.67) (xy 229.87 38.1)
+		)
+		(stroke
+			(width 0)
+			(type default)
+		)
+	)
 	(wire
 		(pts
@@
 	(wire
 		(pts
+			(xy 83.82 26.67) (xy 229.87 26.67)
+		)
+		(stroke
+			(width 0)
+			(type default)
+		)
+	)
+	(wire
+		(pts
 			(xy 204.47 121.92) (xy 204.47 92.71)
 		)
@@
 		)
 		(stroke
+			(width 0)
+			(type default)
+		)
+	)
+	(wire
+		(pts
+			(xy 83.82 39.37) (xy 83.82 26.67)
+		)
+		(stroke

Commit message: Edited footprint
Parts:
- Camera_VSDMini1, Predictor_VSDMini1: symbol VSD:VSDSquadron_mini -> squadron:VSDSquadron_mini
Connections:
- net +3.3V: now also Camera_VSDMini1.20 (+3.3V), Predictor_VSDMini1.20 (+3.3V); no longer Camera_VSDMini1.16 (+3.3V), Predictor_VSDMini1.16 (+3.3V)
- net GND: now also Camera_VSDMini1.21 (GND), Predictor_VSDMini1.21 (GND); no longer Camera_VSDMini1.15 (GND), Predictor_VSDMini1.15 (GND)
- net at Camera_VSDMini1.17 (RX): now also Camera_VSDMini1.28 (Nano_PD5), Predictor_VSDMini1.1 (Nano_PD6)
- net at Predictor_VSDMini1.17 (RX): now also Predictor_VSDMini1.28 (Nano_PD5)
- net at Predictor_VSDMini1.19 (RST): no longer Predictor_VSDMini1.28 (Nano_PD5)
- now unconnected: Camera_VSDMini1.19 (RX)
